Commit message: update zm_robot controller

File: zm_robot_description/urdf/zm_robot.xacro (robot description, xacro)
@@ -29,6 +29,9 @@
   <xacro:property name="roller_9_x" value="0.049792"/>
   <!-- rollor friction -->
-  <xacro:property name="roller_friction" value="0.2"/>
+  <xacro:property name="roller_friction" value="0.4"/>
   <xacro:property name="roller_dampling" value="0"/>
+  <!-- wheel friction -->
+  <xacro:property name="roller_friction_wheel" value="0.2"/>
+  <xacro:property name="roller_dampling_wheel" value="1.5"/>
   <!-- Import all Gazebo-customization elements, including Gazebo colors -->
   <xacro:include filename="$(find zm_robot_description)/urdf/zm_robot.gazebo" />
@@ -36,8 +39,8 @@
   <xacro:include filename="$(find zm_robot_description)/urdf/materials.xacro" />
   <!-- Import rollor actuator -->
-  <xacro:include filename="$(find zm_robot_description)/urdf/rollor_1.gazebo" />
-  <xacro:include filename="$(find zm_robot_description)/urdf/rollor_2.gazebo" />
-  <xacro:include filename="$(find zm_robot_description)/urdf/rollor_3.gazebo" />
-  <xacro:include filename="$(find zm_robot_description)/urdf/rollor_4.gazebo" />
+  <!--xacro:include filename="$(find zm_robot_description)/urdf/rollor_1.gazebo" /-->
+  <!--xacro:include filename="$(find zm_robot_description)/urdf/rollor_2.gazebo" /-->
+  <!--xacro:include filename="$(find zm_robot_description)/urdf/rollor_3.gazebo" /-->
+  <!--xacro:include filename="$(find zm_robot_description)/urdf/rollor_4.gazebo" /-->
   <!-- Used for fixing robot to Gazebo 'base_link' -->
   <link name="base_footprint"/>
@@ -64,9 +67,9 @@
     <inertial>
       <origin xyz="0 0 0" rpy="0 0 0"/>
-      <mass value="9.987"/>
-      <inertia
-	  ixx="0.297561439" ixy="0.0" ixz="0.0"
-	  iyy="0.655537494" iyz="0.0"
-	  izz="0.892409275"/>
+      <mass value="29.964"/>
+      <inertia
+	  ixx="0.892684320" ixy="0.0" ixz="0.0"
+	  iyy="1.966612482" iyz="0.0"
+	  izz="2.677227828"/>
     </inertial>
   </link>
@@ -77,5 +80,5 @@
     <origin xyz="${wheel_after_L} ${wheel_left_W} 0" rpy="${wheel_rotationx} 0 0"/>
     <axis xyz="0 0 1"/>
-    <dynamics damping="0.3" friction="0.2"/>
+    <dynamics damping="${roller_dampling_wheel}" friction="${roller_friction_wheel}"/>
   </joint>
   <link name="wheel_1">
@@ -387,5 +390,5 @@
     <origin xyz="${wheel_before_L} ${wheel_left_W} 0" rpy="${wheel_rotationx} 0 0"/>
     <axis xyz="0 0 1"/>
-    <dynamics damping="0.3" friction="0.2"/>
+    <dynamics damping="${roller_dampling_wheel}" friction="${roller_friction_wheel}"/>
   </joint>
   <link name="wheel_2">
@@ -697,5 +700,5 @@
     <origin xyz="${wheel_before_L} ${wheel_right_W} 0" rpy="${wheel_rotationx} 0 0"/>
     <axis xyz="0 0 1"/>
-    <dynamics damping="0.3" friction="0.2"/>
+    <dynamics damping="${roller_dampling_wheel}" friction="${roller_friction_wheel}"/>
   </joint>
   <link name="wheel_3">
@@ -1007,5 +1010,5 @@
     <origin xyz="${wheel_after_L} ${wheel_right_W} 0" rpy="${wheel_rotationx} 0 0"/>
     <axis xyz="0 0 1"/>
-    <dynamics damping="0.3" friction="0.2"/>
+    <dynamics damping="${roller_dampling_wheel}" friction="${roller_friction_wheel}"/>
   </joint>
   <link name="wheel_4">
@@ -1311,43 +1314,3 @@
     </inertial>
   </link>
-  <transmission name="tran1">
-    <type>transmission_interface/SimpleTransmission</type>
-    <joint name="wheel_joint1">
-      <hardwareInterface>hardware_interface/EffortJointInterface</hardwareInterface>
-    </joint>
-    <actuator name="motor1">
-      <hardwareInterface>hardware_interface/EffortJointInterface</hardwareInterface>
-      <mechanicalReduction>1</mechanicalReduction>
-    </actuator>
-  </transmission>
-  <transmission name="tran2">
-    <type>transmission_interface/SimpleTransmission</type>
-    <joint name="wheel_joint2">
-      <hardwareInterface>hardware_interface/EffortJointInterface</hardwareInterface>
-    </joint>
-    <actuator name="motor2">
-      <hardwareInterface>hardware_interface/EffortJointInterface</hardwareInterface>
-      <mechanicalReduction>1</mechanicalReduction>
-    </actuator>
-  </transmission>
-  <transmission name="tran3">
-    <type>transmission_interface/SimpleTransmission</type>
-    <joint name="wheel_joint3">
-      <hardwareInterface>hardware_interface/EffortJointInterface</hardwareInterface>
-    </joint>
-    <actuator name="motor3">
-      <hardwareInterface>hardware_interface/EffortJointInterface</hardwareInterface>
-      <mechanicalReduction>1</mechanicalReduction>
-    </actuator>
-  </transmission>
-  <transmission name="tran4">
-    <type>transmission_interface/SimpleTransmission</type>
-    <joint name="wheel_joint4">
-      <hardwareInterface>hardware_interface/EffortJointInterface</hardwareInterface>
-    </joint>
-    <actuator name="motor4">
-      <hardwareInterface>hardware_interface/EffortJointInterface</hardwareInterface>
-      <mechanicalReduction>1</mechanicalReduction>
-    </actuator>
-  </transmission>
 </robot>

Commit message: finished zm_robot.

File: zm_robot_description/urdf/zm_robot.xacro (robot description, xacro)
@@ -106,5 +106,5 @@
   </link>
   <!-- roller_1_1 -->
-  <joint name="roller_1_1_joint" type="continuous">
+  <joint name="roller_1_1_joint" type="fixed">
     <parent link="wheel_1"/>
     <child link="roller_1_1"/>
@@ -137,5 +137,5 @@
   </link>
   <!-- roller_1_2 -->
-  <joint name="roller_1_2_joint" type="continuous">
+  <joint name="roller_1_2_joint" type="fixed">
     <parent link="wheel_1"/>
     <child link="roller_1_2"/>
@@ -168,5 +168,5 @@
   </link>
   <!-- roller_1_3 -->
-  <joint name="roller_1_3_joint" type="continuous">
+  <joint name="roller_1_3_joint" type="fixed">
     <parent link="wheel_1"/>
     <child link="roller_1_3"/>
@@ -199,5 +199,5 @@
   </link>
   <!-- roller_1_4 -->
-  <joint name="roller_1_4_joint" type="continuous">
+  <joint name="roller_1_4_joint" type="fixed">
     <parent link="wheel_1"/>
     <child link="roller_1_4"/>
@@ -230,5 +230,5 @@
   </link>
   <!-- roller_1_5 -->
-  <joint name="roller_1_5_joint" type="continuous">
+  <joint name="roller_1_5_joint" type="fixed">
     <parent link="wheel_1"/>
     <child link="roller_1_5"/>
@@ -261,5 +261,5 @@
   </link>
   <!-- roller_1_6 -->
-  <joint name="roller_1_6_joint" type="continuous">
+  <joint name="roller_1_6_joint" type="fixed">
     <parent link="wheel_1"/>
     <child link="roller_1_6"/>
@@ -292,5 +292,5 @@
   </link>
   <!-- roller_1_7 -->
-  <joint name="roller_1_7_joint" type="continuous">
+  <joint name="roller_1_7_joint" type="fixed">
     <parent link="wheel_1"/>
     <child link="roller_1_7"/>
@@ -323,5 +323,5 @@
   </link>
   <!-- roller_1_8 -->
-  <joint name="roller_1_8_joint" type="continuous">
+  <joint name="roller_1_8_joint" type="fixed">
     <parent link="wheel_1"/>
     <child link="roller_1_8"/>
@@ -354,5 +354,5 @@
   </link>
   <!-- roller_1_9 -->
-  <joint name="roller_1_9_joint" type="continuous">
+  <joint name="roller_1_9_joint" type="fixed">
     <parent link="wheel_1"/>
     <child link="roller_1_9"/>
@@ -416,5 +416,5 @@
   </link>
   <!-- roller_2_1 -->
-  <joint name="roller_2_1_joint" type="continuous">
+  <joint name="roller_2_1_joint" type="fixed">
     <parent link="wheel_2"/>
     <child link="roller_2_1"/>
@@ -447,5 +447,5 @@
   </link>
   <!-- roller_2_2 -->
-  <joint name="roller_2_2_joint" type="continuous">
+  <joint name="roller_2_2_joint" type="fixed">
     <parent link="wheel_2"/>
     <child link="roller_2_2"/>
@@ -478,5 +478,5 @@
   </link>
   <!-- roller_2_3 -->
-  <joint name="roller_2_3_joint" type="continuous">
+  <joint name="roller_2_3_joint" type="fixed">
     <parent link="wheel_2"/>
     <child link="roller_2_3"/>
@@ -509,5 +509,5 @@
   </link>
   <!-- roller_2_4 -->
-  <joint name="roller_2_4_joint" type="continuous">
+  <joint name="roller_2_4_joint" type="fixed">
     <parent link="wheel_2"/>
     <child link="roller_2_4"/>
@@ -540,5 +540,5 @@
   </link>
   <!-- roller_2_5 -->
-  <joint name="roller_2_5_joint" type="continuous">
+  <joint name="roller_2_5_joint" type="fixed">
     <parent link="wheel_2"/>
     <child link="roller_2_5"/>
@@ -571,5 +571,5 @@
   </link>
   <!-- roller_2_6 -->
-  <joint name="roller_2_6_joint" type="continuous">
+  <joint name="roller_2_6_joint" type="fixed">
     <parent link="wheel_2"/>
     <child link="roller_2_6"/>
@@ -602,5 +602,5 @@
   </link>
   <!-- roller_2_7 -->
-  <joint name="roller_2_7_joint" type="continuous">
+  <joint name="roller_2_7_joint" type="fixed">
     <parent link="wheel_2"/>
     <child link="roller_2_7"/>
@@ -633,5 +633,5 @@
   </link>
   <!-- roller_2_8 -->
-  <joint name="roller_2_8_joint" type="continuous">
+  <joint name="roller_2_8_joint" type="fixed">
     <parent link="wheel_2"/>
     <child link="roller_2_8"/>
@@ -664,5 +664,5 @@
   </link>
   <!-- roller_2_9 -->
-  <joint name="roller_2_9_joint" type="continuous">
+  <joint name="roller_2_9_joint" type="fixed">
     <parent link="wheel_2"/>
     <child link="roller_2_9"/>
@@ -726,5 +726,5 @@
   </link>
   <!-- roller_3_1 -->
-  <joint name="roller_3_1_joint" type="continuous">
+  <joint name="roller_3_1_joint" type="fixed">
     <parent link="wheel_3"/>
     <child link="roller_3_1"/>
@@ -757,5 +757,5 @@
   </link>
   <!-- roller_3_2 -->
-  <joint name="roller_3_2_joint" type="continuous">
+  <joint name="roller_3_2_joint" type="fixed">
     <parent link="wheel_3"/>
     <child link="roller_3_2"/>
@@ -788,5 +788,5 @@
   </link>
   <!-- roller_3_3 -->
-  <joint name="roller_3_3_joint" type="continuous">
+  <joint name="roller_3_3_joint" type="fixed">
     <parent link="wheel_3"/>
     <child link="roller_3_3"/>
@@ -819,5 +819,5 @@
   </link>
   <!-- roller_3_4 -->
-  <joint name="roller_3_4_joint" type="continuous">
+  <joint name="roller_3_4_joint" type="fixed">
     <parent link="wheel_3"/>
     <child link="roller_3_4"/>
@@ -850,5 +850,5 @@
   </link>
   <!-- roller_3_5 -->
-  <joint name="roller_3_5_joint" type="continuous">
+  <joint name="roller_3_5_joint" type="fixed">
     <parent link="wheel_3"/>
     <child link="roller_3_5"/>
@@ -881,5 +881,5 @@
   </link>
   <!-- roller_3_6 -->
-  <joint name="roller_3_6_joint" type="continuous">
+  <joint name="roller_3_6_joint" type="fixed">
     <parent link="wheel_3"/>
     <child link="roller_3_6"/>
@@ -912,5 +912,5 @@
   </link>
   <!-- roller_3_7 -->
-  <joint name="roller_3_7_joint" type="continuous">
+  <joint name="roller_3_7_joint" type="fixed">
     <parent link="wheel_3"/>
     <child link="roller_3_7"/>
@@ -943,5 +943,5 @@
   </link>
   <!-- roller_3_8 -->
-  <joint name="roller_3_8_joint" type="continuous">
+  <joint name="roller_3_8_joint" type="fixed">
     <parent link="wheel_3"/>
     <child link="roller_3_8"/>
@@ -974,5 +974,5 @@
   </link>
   <!-- roller_3_9 -->
-  <joint name="roller_3_9_joint" type="continuous">
+  <joint name="roller_3_9_joint" type="fixed">
     <parent link="wheel_3"/>
     <child link="roller_3_9"/>
@@ -1036,5 +1036,5 @@
   </link>
   <!-- roller_4_1 -->
-  <joint name="roller_4_1_joint" type="continuous">
+  <joint name="roller_4_1_joint" type="fixed">
     <parent link="wheel_4"/>
     <child link="roller_4_1"/>
@@ -1067,5 +1067,5 @@
   </link>
   <!-- roller_4_2 -->
-  <joint name="roller_4_2_joint" type="continuous">
+  <joint name="roller_4_2_joint" type="fixed">
     <parent link="wheel_4"/>
     <child link="roller_4_2"/>
@@ -1098,5 +1098,5 @@
   </link>
   <!-- roller_4_3 -->
-  <joint name="roller_4_3_joint" type="continuous">
+  <joint name="roller_4_3_joint" type="fixed">
     <parent link="wheel_4"/>
     <child link="roller_4_3"/>
@@ -1129,5 +1129,5 @@
   </link>
   <!-- roller_4_4 -->
-  <joint name="roller_4_4_joint" type="continuous">
+  <joint name="roller_4_4_joint" type="fixed">
     <parent link="wheel_4"/>
     <child link="roller_4_4"/>
@@ -1160,5 +1160,5 @@
   </link>
   <!-- roller_4_5 -->
-  <joint name="roller_4_5_joint" type="continuous">
+  <joint name="roller_4_5_joint" type="fixed">
     <parent link="wheel_4"/>
     <child link="roller_4_5"/>
@@ -1191,5 +1191,5 @@
   </link>
   <!-- roller_4_6 -->
-  <joint name="roller_4_6_joint" type="continuous">
+  <joint name="roller_4_6_joint" type="fixed">
     <parent link="wheel_4"/>
     <child link="roller_4_6"/>
@@ -1222,5 +1222,5 @@
   </link>
   <!-- roller_4_7 -->
-  <joint name="roller_4_7_joint" type="continuous">
+  <joint name="roller_4_7_joint" type="fixed">
     <parent link="wheel_4"/>
     <child link="roller_4_7"/>
@@ -1253,5 +1253,5 @@
   </link>
   <!-- roller_4_8 -->
-  <joint name="roller_4_8_joint" type="continuous">
+  <joint name="roller_4_8_joint" type="fixed">
     <parent link="wheel_4"/>
     <child link="roller_4_8"/>
@@ -1284,5 +1284,5 @@
   </link>
   <!-- roller_4_9 -->
-  <joint name="roller_4_9_joint" type="continuous">
+  <joint name="roller_4_9_joint" type="fixed">
     <parent link="wheel_4"/>
     <child link="roller_4_9"/>

Commit message: Add LiDAR and image sensor in urdf file.

File: zm_robot_description/urdf/zm_robot.xacro (robot description, xacro)
@@ -1314,3 +1314,90 @@
     </inertial>
   </link>
+  <!-- sick LiDAR 0 -->
+  <joint name="sick_lidar0_joint" type="fixed">
+    <parent link="base_link"/>
+    <child link="sick_lidar0"/>
+    <origin xyz="0.33 0.175 0.195722" rpy="0 0 0.7854"/>
+  </joint>
+  <link name="sick_lidar0">
+    <collision>
+      <origin xyz="0 0 0" rpy="0 0 0"/>
+      <geometry>
+	<mesh filename="package://zm_robot_description/meshes/sick_s30b.stl" scale="0.01 0.01 0.01"/>
+      </geometry>
+    </collision>
+    <visual>
+      <origin xyz="0 0 0" rpy="0 0 0"/>
+      <geometry>
+	<mesh filename="package://zm_robot_description/meshes/sick_s30b.stl" scale="0.01 0.01 0.01"/>
+      </geometry>
+      <material name="green"/>
+    </visual>
+    <inertial>
+      <origin xyz="0 0 0" rpy="0 0 0"/>
+      <mass value="1.2"/>
+      <inertia
+	  ixx="0.0001" ixy="0.0" ixz="0.0"
+	  iyy="0.0001" iyz="0.0"
+	  izz="0.0001"/>
+    </inertial>
+  </link>
+  <!-- sick LiDAR 1 -->
+  <joint name="sick_lidar1_joint" type="fixed">
+    <parent link="base_link"/>
+    <child link="sick_lidar1"/>
+    <origin xyz="-0.33 -0.175 0.195722" rpy="0 0 -2.35619"/>
+  </joint>
+  <link name="sick_lidar1">
+    <collision>
+      <origin xyz="0 0 0" rpy="0 0 0"/>
+      <geometry>
+	<mesh filename="package://zm_robot_description/meshes/sick_s30b.stl" scale="0.01 0.01 0.01"/>
+      </geometry>
+    </collision>
+    <visual>
+      <origin xyz="0 0 0" rpy="0 0 0"/>
+      <geometry>
+	<mesh filename="package://zm_robot_description/meshes/sick_s30b.stl" scale="0.01 0.01 0.01"/>
+      </geometry>
+      <material name="green"/>
+    </visual>
+    <inertial>
+      <origin xyz="0 0 0" rpy="0 0 0"/>
+      <mass value="1.2"/>
+      <inertia
+	  ixx="0.0001" ixy="0.0" ixz="0.0"
+	  iyy="0.0001" iyz="0.0"
+	  izz="0.0001"/>
+    </inertial>
+  </link>
+  <!-- kinect V2 -->
+  <joint name="kinect_v2_joint " type="fixed">
+    <parent link="base_link"/>
+    <child link="kinect_v2"/>
+    <origin xyz="0.297 -0.05 0.122015" rpy="-1.5708 0 -1.5708"/>
+  </joint>
+  <link name="kinect_v2">
+    <collision>
+      <origin xyz="0 0 0" rpy="0 0 0"/>
+      <geometry>
+	<mesh filename="package://zm_robot_description/meshes/kinect_v2.stl" scale="0.01 0.01 0.01"/>
+      </geometry>
+    </collision>
+    <visual>
+      <origin xyz="0 0 0" rpy="0 0 0"/>
+      <geometry>
+	<mesh filename="package://zm_robot_description/meshes/kinect_v2.stl" scale="0.01 0.01 0.01"/>
+      </geometry>
+      <material name="black"/>
+    </visual>
+    <inertial>
+      <origin xyz="0 0 0" rpy="0 0 0"/>
+      <mass value="0.5"/>
+      <inertia
+	  ixx="0.00005" ixy="0.0" ixz="0.0"
+	  iyy="0.00005" iyz="0.0"
+	  izz="0.00005"/>
+    </inertial>
+  </link>
 </robot>

File: zm_robot_description/urdf/zm_robot_pid.xacro (robot description, xacro)
@@ -1314,3 +1314,90 @@
     </inertial>
   </link>
+  <!-- sick LiDAR 0 -->
+  <joint name="sick_lidar0_joint" type="fixed">
+    <parent link="base_link"/>
+    <child link="sick_lidar0"/>
+    <origin xyz="0.33 0.175 0.195722" rpy="0 0 0.7854"/>
+  </joint>
+  <link name="sick_lidar0">
+    <collision>
+      <origin xyz="0 0 0" rpy="0 0 0"/>
+      <geometry>
+	<mesh filename="package://zm_robot_description/meshes/sick_s30b.stl" scale="0.01 0.01 0.01"/>
+      </geometry>
+    </collision>
+    <visual>
+      <origin xyz="0 0 0" rpy="0 0 0"/>
+      <geometry>
+	<mesh filename="package://zm_robot_description/meshes/sick_s30b.stl" scale="0.01 0.01 0.01"/>
+      </geometry>
+      <material name="green"/>
+    </visual>
+    <inertial>
+      <origin xyz="0 0 0" rpy="0 0 0"/>
+      <mass value="1.2"/>
+      <inertia
+	  ixx="0.0001" ixy="0.0" ixz="0.0"
+	  iyy="0.0001" iyz="0.0"
+	  izz="0.0001"/>
+    </inertial>
+  </link>
+  <!-- sick LiDAR 1 -->
+  <joint name="sick_lidar1_joint" type="fixed">
+    <parent link="base_link"/>
+    <child link="sick_lidar1"/>
+    <origin xyz="-0.33 -0.175 0.195722" rpy="0 0 -2.35619"/>
+  </joint>
+  <link name="sick_lidar1">
+    <collision>
+      <origin xyz="0 0 0" rpy="0 0 0"/>
+      <geometry>
+	<mesh filename="package://zm_robot_description/meshes/sick_s30b.stl" scale="0.01 0.01 0.01"/>
+      </geometry>
+    </collision>
+    <visual>
+      <origin xyz="0 0 0" rpy="0 0 0"/>
+      <geometry>
+	<mesh filename="package://zm_robot_description/meshes/sick_s30b.stl" scale="0.01 0.01 0.01"/>
+      </geometry>
+      <material name="green"/>
+    </visual>
+    <inertial>
+      <origin xyz="0 0 0" rpy="0 0 0"/>
+      <mass value="1.2"/>
+      <inertia
+	  ixx="0.0001" ixy="0.0" ixz="0.0"
+	  iyy="0.0001" iyz="0.0"
+	  izz="0.0001"/>
+    </inertial>
+  </link>
+  <!-- kinect V2 -->
+  <joint name="kinect_v2_joint " type="fixed">
+    <parent link="base_link"/>
+    <child link="kinect_v2"/>
+    <origin xyz="0.297 -0.05 0.122015" rpy="-1.5708 0 -1.5708"/>
+  </joint>
+  <link name="kinect_v2">
+    <collision>
+      <origin xyz="0 0 0" rpy="0 0 0"/>
+      <geometry>
+	<mesh filename="package://zm_robot_description/meshes/kinect_v2.stl" scale="0.01 0.01 0.01"/>
+      </geometry>
+    </collision>
+    <visual>
+      <origin xyz="0 0 0" rpy="0 0 0"/>
+      <geometry>
+	<mesh filename="package://zm_robot_description/meshes/kinect_v2.stl" scale="0.01 0.01 0.01"/>
+      </geometry>
+      <material name="black"/>
+    </visual>
+    <inertial>
+      <origin xyz="0 0 0" rpy="0 0 0"/>
+      <mass value="0.5"/>
+      <inertia
+	  ixx="0.00005" ixy="0.0" ixz="0.0"
+	  iyy="0.00005" iyz="0.0"
+	  izz="0.00005"/>
+    </inertial>
+  </link>
 </robot>

Commit message: revised zm_robot controller and added landscape.

File: zm_robot_description/urdf/zm_robot.xacro (robot description, xacro)
@@ -1377,4 +1377,5 @@
     <child link="kinect_v2"/>
     <origin xyz="0.297 -0.05 0.122015" rpy="-1.5708 0 -1.5708"/>
+    <axis xyz="0 0 1"/>
   </joint>
   <link name="kinect_v2">

File: zm_robot_description/urdf/zm_robot_pid.xacro (robot description, xacro)
@@ -1377,4 +1377,5 @@
     <child link="kinect_v2"/>
     <origin xyz="0.297 -0.05 0.122015" rpy="-1.5708 0 -1.5708"/>
+    <axis xyz="0 0 1"/>
   </joint>
   <link name="kinect_v2">

Commit message: Add IMU sensor controller and revised Kinect V2.

File: zm_robot_description/urdf/zm_robot.xacro (robot description, xacro)
@@ -1376,5 +1376,5 @@
     <parent link="base_link"/>
     <child link="kinect_v2"/>
-    <origin xyz="0.297 -0.05 0.122015" rpy="-1.5708 0 -1.5708"/>
+    <origin xyz="0.297 -0.05 0.122015" rpy="0 0 0"/>
     <axis xyz="0 0 1"/>
   </joint>
@@ -1402,3 +1402,33 @@
     </inertial>
   </link>
+  <!-- IMU -->
+  <joint name="IMU_joint " type="fixed">
+    <parent link="base_link"/>
+    <child link="IMU_sensor"/>
+    <origin xyz="0 0 0.08" rpy="0 0 0"/>
+    <axis xyz="0 0 1"/>
+  </joint>
+  <link name="IMU_sensor">
+    <collision>
+      <origin xyz="0 0 0" rpy="0 0 0"/>
+      <geometry>
+	<mesh filename="package://zm_robot_description/meshes/IMU_sensor.stl" scale="0.01 0.01 0.01"/>
+      </geometry>
+    </collision>
+    <visual>
+      <origin xyz="0 0 0" rpy="0 0 0"/>
+      <geometry>
+	<mesh filename="package://zm_robot_description/meshes/IMU_sensor.stl" scale="0.01 0.01 0.01"/>
+      </geometry>
+      <material name="red"/>
+    </visual>
+    <inertial>
+      <origin xyz="0 0 0" rpy="0 0 0"/>
+      <mass value="0.5"/>
+      <inertia
+	  ixx="0.00005" ixy="0.0" ixz="0.0"
+	  iyy="0.00005" iyz="0.0"
+	  izz="0.00005"/>
+    </inertial>
+  </link>
 </robot>

File: zm_robot_description/urdf/zm_robot_pid.xacro (robot description, xacro)
@@ -1376,5 +1376,5 @@
     <parent link="base_link"/>
     <child link="kinect_v2"/>
-    <origin xyz="0.297 -0.05 0.122015" rpy="-1.5708 0 -1.5708"/>
+    <origin xyz="0.297 -0.05 0.122015" rpy="0 0 0"/>
     <axis xyz="0 0 1"/>
   </joint>
@@ -1402,3 +1402,33 @@
     </inertial>
   </link>
+  <!-- IMU -->
+  <joint name="IMU_joint " type="fixed">
+    <parent link="base_link"/>
+    <child link="IMU_sensor"/>
+    <origin xyz="0 0 0.08" rpy="0 0 0"/>
+    <axis xyz="0 0 1"/>
+  </joint>
+  <link name="IMU_sensor">
+    <collision>
+      <origin xyz="0 0 0" rpy="0 0 0"/>
+      <geometry>
+	<mesh filename="package://zm_robot_description/meshes/IMU_sensor.stl" scale="0.01 0.01 0.01"/>
+      </geometry>
+    </collision>
+    <visual>
+      <origin xyz="0 0 0" rpy="0 0 0"/>
+      <geometry>
+	<mesh filename="package://zm_robot_description/meshes/IMU_sensor.stl" scale="0.01 0.01 0.01"/>
+      </geometry>
+      <material name="red"/>
+    </visual>
+    <inertial>
+      <origin xyz="0 0 0" rpy="0 0 0"/>
+      <mass value="0.5"/>
+      <inertia
+	  ixx="0.00005" ixy="0.0" ixz="0.0"
+	  iyy="0.00005" iyz="0.0"
+	  izz="0.00005"/>
+    </inertial>
+  </link>
 </robot>
