Commit message: Add files via upload

File: zm_robot_description/urdf/zm_robot_wheel_LF.urdf.xacro (robot description, xacro)
@@ -25,6 +25,6 @@
           <origin xyz="0.001 0 0" rpy="0 0 0"/>
           <mass value="1.7"/>
-          <inertia ixx="0.004248052" ixy="0.0" ixz="0.0"
-	               iyy="0.004248045" iyz="0.0" izz="0.004879970"/>
+          <inertia ixx="0.04248052" ixy="0.0" ixz="0.0"
+	               iyy="0.04248045" iyz="0.0" izz="0.04879970"/>
       </inertial>
 	</link>

File: zm_robot_description/urdf/zm_robot_wheel_LR.urdf.xacro (robot description, xacro)
@@ -25,6 +25,6 @@
           <origin xyz="0.001 0 0" rpy="0 0 0"/>
           <mass value="1.7"/>
-          <inertia ixx="0.004248052" ixy="0.0" ixz="0.0"
-	               iyy="0.004248045" iyz="0.0" izz="0.004879970"/>
+          <inertia ixx="0.04248052" ixy="0.0" ixz="0.0"
+	               iyy="0.04248045" iyz="0.0" izz="0.04879970"/>
       </inertial>
 	</link>

File: zm_robot_description/urdf/zm_robot_wheel_RF.urdf.xacro (robot description, xacro)
@@ -25,6 +25,6 @@
           <origin xyz="-0.001 0 0" rpy="0 0 0"/>
           <mass value="1.7"/>
-          <inertia ixx="0.004248052" ixy="0.0" ixz="0.0"
-	               iyy="0.004248045" iyz="0.0" izz="-0.004879970"/>
+          <inertia ixx="0.04248052" ixy="0.0" ixz="0.0"
+	               iyy="0.04248045" iyz="0.0" izz="-0.04879970"/>
       </inertial>
 	</link>

File: zm_robot_description/urdf/zm_robot_wheel_RR.urdf.xacro (robot description, xacro)
@@ -25,6 +25,6 @@
           <origin xyz="-0.001 0 0" rpy="0 0 0"/>
           <mass value="1.7"/>
-          <inertia ixx="0.004248052" ixy="0.0" ixz="0.0"
-	               iyy="0.004248045" iyz="0.0" izz="-0.004879970"/>
+          <inertia ixx="0.04248052" ixy="0.0" ixz="0.0"
+	               iyy="0.04248045" iyz="0.0" izz="-0.04879970"/>
       </inertial>
 	</link>
