Commit message: zm robot ros2

File: zm_robot_description/urdf/zm_robot.urdf.xacro (robot description, xacro)
@@ -38,5 +38,4 @@
   <!-- Import Plugin -->
   <xacro:include filename="$(find zm_robot_description)/urdf/zm_robot_plugin.gazebo"/>
-  <!--xacro:include filename="$(find zm_robot_description)/urdf/zm_robot_plugin.gazebo"/-->
   <!-- Used for fixing robot to Gazebo 'base_link' -->
   <link name="base_footprint"/>
@@ -51,11 +50,11 @@
       <origin xyz="0 0 0" rpy="0 0 0"/>
       <geometry>
-        <mesh filename="package://zm_robot_description/meshes/agv_base.stl" scale="0.01 0.01 0.01"/>
-      </geometry>
-    </collision>
-    <visual>
-      <origin xyz="0 0 0" rpy="0 0 0"/>
-      <geometry>
-        <mesh filename="package://zm_robot_description/meshes/agv_base.stl" scale="0.01 0.01 0.01"/>
+        <mesh filename="file://$(find zm_robot_description)/meshes/agv_base.stl" scale="0.01 0.01 0.01"/>
+      </geometry>
+    </collision>
+    <visual>
+      <origin xyz="0 0 0" rpy="0 0 0"/>
+      <geometry>
+        <mesh filename="file://$(find zm_robot_description)/meshes/agv_base.stl" scale="0.01 0.01 0.01"/>
       </geometry>
       <material name="orange"/>
@@ -79,11 +78,11 @@
       <origin xyz="0 0 0" rpy="0 0 0"/>
       <geometry>
-        <mesh filename="package://zm_robot_description/meshes/sick_s30b.stl" scale="0.01 0.01 0.01"/>
-      </geometry>
-    </collision>
-    <visual>
-      <origin xyz="0 0 0" rpy="0 0 0"/>
-      <geometry>
-        <mesh filename="package://zm_robot_description/meshes/sick_s30b.stl" scale="0.01 0.01 0.01"/>
+        <mesh filename="file://$(find zm_robot_description)/meshes/sick_s30b.stl" scale="0.01 0.01 0.01"/>
+      </geometry>
+    </collision>
+    <visual>
+      <origin xyz="0 0 0" rpy="0 0 0"/>
+      <geometry>
+        <mesh filename="file://$(find zm_robot_description)/meshes/sick_s30b.stl" scale="0.01 0.01 0.01"/>
       </geometry>
       <material name="green"/>
@@ -107,11 +106,11 @@
       <origin xyz="0 0 0" rpy="0 0 0"/>
       <geometry>
-        <mesh filename="package://zm_robot_description/meshes/sick_s30b.stl" scale="0.01 0.01 0.01"/>
-      </geometry>
-    </collision>
-    <visual>
-      <origin xyz="0 0 0" rpy="0 0 0"/>
-      <geometry>
-        <mesh filename="package://zm_robot_description/meshes/sick_s30b.stl" scale="0.01 0.01 0.01"/>
+        <mesh filename="file://$(find zm_robot_description)/meshes/sick_s30b.stl" scale="0.01 0.01 0.01"/>
+      </geometry>
+    </collision>
+    <visual>
+      <origin xyz="0 0 0" rpy="0 0 0"/>
+      <geometry>
+        <mesh filename="file://$(find zm_robot_description)/meshes/sick_s30b.stl" scale="0.01 0.01 0.01"/>
       </geometry>
       <material name="green"/>
@@ -136,11 +135,11 @@
       <origin xyz="0 0 0" rpy="0 0 0"/>
       <geometry>
-	      <mesh filename="package://zm_robot_description/meshes/kinect_v2.stl" scale="0.01 0.01 0.01"/>
-      </geometry>
-    </collision>
-    <visual>
-      <origin xyz="0 0 0" rpy="0 0 0"/>
-      <geometry>
-	      <mesh filename="package://zm_robot_description/meshes/kinect_v2.stl" scale="0.01 0.01 0.01"/>
+	      <mesh filename="file://$(find zm_robot_description)/meshes/kinect_v2.stl" scale="0.01 0.01 0.01"/>
+      </geometry>
+    </collision>
+    <visual>
+      <origin xyz="0 0 0" rpy="0 0 0"/>
+      <geometry>
+	      <mesh filename="file://$(find zm_robot_description)/meshes/kinect_v2.stl" scale="0.01 0.01 0.01"/>
       </geometry>
       <material name="black"/>
@@ -165,11 +164,11 @@
       <origin xyz="0 0 0" rpy="0 0 0"/>
       <geometry>
-	      <mesh filename="package://zm_robot_description/meshes/IMU_sensor.stl" scale="0.01 0.01 0.01"/>
-      </geometry>
-    </collision>
-    <visual>
-      <origin xyz="0 0 0" rpy="0 0 0"/>
-      <geometry>
-	      <mesh filename="package://zm_robot_description/meshes/IMU_sensor.stl" scale="0.01 0.01 0.01"/>
+	      <mesh filename="file://$(find zm_robot_description)/meshes/IMU_sensor.stl" scale="0.01 0.01 0.01"/>
+      </geometry>
+    </collision>
+    <visual>
+      <origin xyz="0 0 0" rpy="0 0 0"/>
+      <geometry>
+	      <mesh filename="file://$(find zm_robot_description)/meshes/IMU_sensor.stl" scale="0.01 0.01 0.01"/>
       </geometry>
       <material name="red"/>

File: zm_robot_description/urdf/zm_robot_wheel_LF.urdf.xacro (robot description, xacro)
@@ -13,5 +13,5 @@
 	  <visual>
 		<geometry>
-		  <mesh filename="package://zm_robot_description/meshes/mecanum_left_before.stl" scale="0.01 0.01 0.01"/>
+		  <mesh filename="file://$(find zm_robot_description)/meshes/mecanum_left_before.stl" scale="0.01 0.01 0.01"/>
 		</geometry>
 		<material name="white"/>
@@ -19,5 +19,5 @@
 	  <collision>
 		<geometry>
-		  <mesh filename="package://zm_robot_description/meshes/mecanum_left_before.stl" scale="0.01 0.01 0.01"/>
+		  <mesh filename="file://$(find zm_robot_description)/meshes/mecanum_left_before.stl" scale="0.01 0.01 0.01"/>
 		</geometry>
 	  </collision>

File: zm_robot_description/urdf/zm_robot_wheel_LR.urdf.xacro (robot description, xacro)
@@ -13,5 +13,5 @@
 	  <visual>
 		<geometry>
-		  <mesh filename="package://zm_robot_description/meshes/mecanum_left_after.stl" scale="0.01 0.01 0.01"/>
+		  <mesh filename="file://$(find zm_robot_description)/meshes/mecanum_left_after.stl" scale="0.01 0.01 0.01"/>
 		</geometry>
 		<material name="white"/>
@@ -19,5 +19,5 @@
 	  <collision>
 		<geometry>
-		  <mesh filename="package://zm_robot_description/meshes/mecanum_left_after.stl" scale="0.01 0.01 0.01"/>
+		  <mesh filename="file://$(find zm_robot_description)/meshes/mecanum_left_after.stl" scale="0.01 0.01 0.01"/>
 		</geometry>
 	  </collision>

File: zm_robot_description/urdf/zm_robot_wheel_RF.urdf.xacro (robot description, xacro)
@@ -13,5 +13,5 @@
 	  <visual>
 		<geometry>
-		  <mesh filename="package://zm_robot_description/meshes/mecanum_right_before.stl" scale="0.01 0.01 0.01"/>
+		  <mesh filename="file://$(find zm_robot_description)/meshes/mecanum_right_before.stl" scale="0.01 0.01 0.01"/>
 		</geometry>
 		<material name="white"/>
@@ -19,5 +19,5 @@
 	  <collision>
 		<geometry>
-		  <mesh filename="package://zm_robot_description/meshes/mecanum_right_before.stl" scale="0.01 0.01 0.01"/>
+		  <mesh filename="file://$(find zm_robot_description)/meshes/mecanum_right_before.stl" scale="0.01 0.01 0.01"/>
 		</geometry>
 	  </collision>

File: zm_robot_description/urdf/zm_robot_wheel_RR.urdf.xacro (robot description, xacro)
@@ -13,5 +13,5 @@
 	  <visual>
 		<geometry>
-		  <mesh filename="package://zm_robot_description/meshes/mecanum_right_after.stl" scale="0.01 0.01 0.01"/>
+		  <mesh filename="file://$(find zm_robot_description)/meshes/mecanum_right_after.stl" scale="0.01 0.01 0.01"/>
 		</geometry>
 		<material name="white"/>
@@ -19,5 +19,5 @@
 	  <collision>
 		<geometry>
-		  <mesh filename="package://zm_robot_description/meshes/mecanum_right_after.stl" scale="0.01 0.01 0.01"/>
+		  <mesh filename="file://$(find zm_robot_description)/meshes/mecanum_right_after.stl" scale="0.01 0.01 0.01"/>
 		</geometry>
 	  </collision>

Commit message: zm_robot add 4 ultrasound sensor and plugin.

File: zm_robot_description/urdf/zm_robot.urdf.xacro (robot description, xacro)
@@ -9,4 +9,16 @@
   <xacro:property name="wheel_left_W" value="0.3" /> <!-- wheel left W -->
   <xacro:property name="wheel_right_W" value="-0.3" /> <!-- wheel right W -->
+  <!-- ultrasound position on robot-->
+  <xacro:property name="ul_left_front_x" value="0.4"/>
+  <xacro:property name="ul_left_front_y" value="0.15" />
+  <xacro:property name="ul_right_front_x" value="0.4" />
+  <xacro:property name="ul_right_front_y" value="-0.15" />
+  <xacro:property name="ul_left_rear_x" value="-0.4" />
+  <xacro:property name="ul_left_rear_y" value="0.15" />
+  <xacro:property name="ul_right_rear_x" value="-0.4" />
+  <xacro:property name="ul_right_rear_y" value="-0.15" />
+  <xacro:property name="ul_hight" value="0.03" />
+  <xacro:property name="ul_front_rotation" value="0" />
+  <xacro:property name="ul_rear_rotation" value="3.141592654" />
   <!-- roller position -->
   <xacro:property name="roller_1_y" value="0"/>
@@ -36,4 +48,6 @@
   <xacro:include filename="$(find zm_robot_description)/urdf/zm_robot_wheel_RF.urdf.xacro"/>
   <xacro:include filename="$(find zm_robot_description)/urdf/zm_robot_wheel_RR.urdf.xacro"/>
+  <!-- Import Ultrasound -->
+  <xacro:include filename="$(find zm_robot_description)/urdf/zm_robot_ultrasound.urdf.xacro"/>
   <!-- Import Plugin -->
   <xacro:include filename="$(find zm_robot_description)/urdf/zm_robot_plugin.gazebo"/>
@@ -386,3 +400,16 @@
   <xacro:roller_trans_v0 prefix="roller_4_8"/>
   <xacro:roller_trans_v0 prefix="roller_4_9"/>
+  <!-- ultrasound -->
+  <xacro:zm_ultrasound prefix="1" parent="base_link" origin_x="${ul_left_front_x}" origin_y="${ul_left_front_y}"
+                                                     origin_z="${ul_hight}" rotation_z="${ul_front_rotation}">
+  </xacro:zm_ultrasound>
+  <xacro:zm_ultrasound prefix="2" parent="base_link" origin_x="${ul_right_front_x}" origin_y="${ul_right_front_y}"
+                                                     origin_z="${ul_hight}" rotation_z="${ul_front_rotation}">
+  </xacro:zm_ultrasound>
+  <xacro:zm_ultrasound prefix="3" parent="base_link" origin_x="${ul_left_rear_x}" origin_y="${ul_left_rear_y}"
+                                                     origin_z="${ul_hight}" rotation_z="${ul_rear_rotation}">
+  </xacro:zm_ultrasound>
+  <xacro:zm_ultrasound prefix="4" parent="base_link" origin_x="${ul_right_rear_x}" origin_y="${ul_right_rear_y}"
+                                                     origin_z="${ul_hight}" rotation_z="${ul_rear_rotation}">
+  </xacro:zm_ultrasound>
 </robot>

File: zm_robot_description/urdf/zm_robot_ultrasound.urdf.xacro (robot description, xacro)
@@ -2,9 +2,9 @@
 <robot xmlns:xacro="http://ros.org/wiki/xacro">
   <xacro:include filename="$(find zm_robot_description)/urdf/zm_robot_ultrasound.gazebo"/>
-  <xacro:macro name="zm_ultrasound" params="prefix parent origin_x origin_y rotation_x">
+  <xacro:macro name="zm_ultrasound" params="prefix parent origin_x origin_y origin_z rotation_z">
 	<joint name="ultrasound_joint_${prefix}" type="fixed">
 	  <parent link="${parent}"/>
 	  <child link="ultrasound_${prefix}"/>
-	  <origin xyz="${origin_x} ${origin_y} 0" rpy="${rotation_x} 0 0"/>
+	  <origin xyz="${origin_x} ${origin_y} ${origin_z}" rpy="0 0 ${rotation_z}"/>
       <axis xyz="0 0 1"/>
 	  <dynamics damping="3.0" friction="5.0"/>
@@ -13,5 +13,5 @@
 	  <visual>
 		<geometry>
-		  <mesh filename="package://zm_robot_description/meshes/ultrasound.stl" scale="0.01 0.01 0.01"/>
+		  <mesh filename="package://zm_robot_description/meshes/ultrasound.stl" scale="0.1 0.1 0.1"/>
 		</geometry>
 		<material name="blue"/>
@@ -19,5 +19,5 @@
 	  <collision>
 		<geometry>
-		  <mesh filename="package://zm_robot_description/meshes/ultrasound.stl" scale="0.01 0.01 0.01"/>
+		  <mesh filename="package://zm_robot_description/meshes/ultrasound.stl" scale="0.1 0.1 0.1"/>
 		</geometry>
 	  </collision>

Commit message: Add 4 ultrasound sensor.

File: zm_robot_description/urdf/zm_robot.urdf.xacro (robot description, xacro)
@@ -9,4 +9,16 @@
   <xacro:property name="wheel_left_W" value="0.3" /> <!-- wheel left W -->
   <xacro:property name="wheel_right_W" value="-0.3" /> <!-- wheel right W -->
+  <!-- ultrasound position on robot-->
+  <xacro:property name="ul_left_front_x" value="0.4"/>
+  <xacro:property name="ul_left_front_y" value="0.15" />
+  <xacro:property name="ul_right_front_x" value="0.4" />
+  <xacro:property name="ul_right_front_y" value="-0.15" />
+  <xacro:property name="ul_left_rear_x" value="-0.4" />
+  <xacro:property name="ul_left_rear_y" value="0.15" />
+  <xacro:property name="ul_right_rear_x" value="-0.4" />
+  <xacro:property name="ul_right_rear_y" value="-0.15" />
+  <xacro:property name="ul_hight" value="0.03" />
+  <xacro:property name="ul_front_rotation" value="0" />
+  <xacro:property name="ul_rear_rotation" value="3.141592654" />
   <!-- roller position -->
   <xacro:property name="roller_1_y" value="0"/>
@@ -36,4 +48,6 @@
   <xacro:include filename="$(find zm_robot_description)/urdf/zm_robot_wheel_RF.urdf.xacro"/>
   <xacro:include filename="$(find zm_robot_description)/urdf/zm_robot_wheel_RR.urdf.xacro"/>
+  <!-- Import Ultrasound -->
+  <xacro:include filename="$(find zm_robot_description)/urdf/zm_robot_ultrasound.urdf.xacro"/>
   <!-- Import Plugin -->
   <xacro:include filename="$(find zm_robot_description)/urdf/zm_robot_plugin.gazebo"/>
@@ -385,3 +399,16 @@
   <xacro:roller_trans_v0 prefix="roller_4_8"/>
   <xacro:roller_trans_v0 prefix="roller_4_9"/>
+  <!-- ultrasound -->
+  <xacro:zm_ultrasound prefix="1" parent="base_link" origin_x="${ul_left_front_x}" origin_y="${ul_left_front_y}"
+                                                     origin_z="${ul_hight}" rotation_z="${ul_front_rotation}">
+  </xacro:zm_ultrasound>
+  <xacro:zm_ultrasound prefix="2" parent="base_link" origin_x="${ul_right_front_x}" origin_y="${ul_right_front_y}"
+                                                     origin_z="${ul_hight}" rotation_z="${ul_front_rotation}">
+  </xacro:zm_ultrasound>
+  <xacro:zm_ultrasound prefix="3" parent="base_link" origin_x="${ul_left_rear_x}" origin_y="${ul_left_rear_y}"
+                                                     origin_z="${ul_hight}" rotation_z="${ul_rear_rotation}">
+  </xacro:zm_ultrasound>
+  <xacro:zm_ultrasound prefix="4" parent="base_link" origin_x="${ul_right_rear_x}" origin_y="${ul_right_rear_y}"
+                                                     origin_z="${ul_hight}" rotation_z="${ul_rear_rotation}">
+  </xacro:zm_ultrasound>
 </robot>

Commit message: Update Gazebo.

File: zm_robot_description/urdf/zm_robot.urdf.xacro (robot description, xacro)
@@ -50,6 +50,4 @@
   <!-- Import Ultrasound -->
   <xacro:include filename="$(find zm_robot_description)/urdf/zm_robot_ultrasound.urdf.xacro"/>
-  <!-- Import Plugin -->
-  <!--xacro:include filename="$(find zm_robot_description)/urdf/zm_robot_plugin.gazebo"/-->
   <!-- Used for fixing robot to Gazebo 'base_link' -->
   <link name="base_footprint"/>
@@ -108,5 +106,5 @@
 	             iyy="0.0001" iyz="0.0"
 	             izz="0.0001"/>
-      </inertial>
+    </inertial>
   </link>
   <!-- sick LiDAR 1 -->
@@ -136,5 +134,5 @@
 	             iyy="0.0001" iyz="0.0"
 	             izz="0.0001"/>
-      </inertial>
+    </inertial>
   </link>
   <!-- kinect V2 -->

Commit message: Remap frame id in gazebo.

File: zm_robot_description/urdf/zm_robot.urdf.xacro (robot description, xacro)
@@ -322,83 +322,4 @@
                                                            rotation_x="-0.7854" rotation_z="-0.6981">
   </xacro:zm_roller_v0>
-  <!-- Wheel -->
-  <xacro:wheel_gazebo_v0 prefix="1"/>
-  <xacro:wheel_gazebo_v0 prefix="2"/>
-  <xacro:wheel_gazebo_v0 prefix="3"/>
-  <xacro:wheel_gazebo_v0 prefix="4"/>
-  <!-- Rollor -->
-  <xacro:roller_gazebo_v0 prefix="roller_1_1"/>
-  <xacro:roller_gazebo_v0 prefix="roller_1_2"/>
-  <xacro:roller_gazebo_v0 prefix="roller_1_3"/>
-  <xacro:roller_gazebo_v0 prefix="roller_1_4"/>
-  <xacro:roller_gazebo_v0 prefix="roller_1_5"/>
-  <xacro:roller_gazebo_v0 prefix="roller_1_6"/>
-  <xacro:roller_gazebo_v0 prefix="roller_1_7"/>
-  <xacro:roller_gazebo_v0 prefix="roller_1_8"/>
-  <xacro:roller_gazebo_v0 prefix="roller_1_9"/>
-  <xacro:roller_gazebo_v0 prefix="roller_2_1"/>
-  <xacro:roller_gazebo_v0 prefix="roller_2_2"/>
-  <xacro:roller_gazebo_v0 prefix="roller_2_3"/>
-  <xacro:roller_gazebo_v0 prefix="roller_2_4"/>
-  <xacro:roller_gazebo_v0 prefix="roller_2_5"/>
-  <xacro:roller_gazebo_v0 prefix="roller_2_6"/>
-  <xacro:roller_gazebo_v0 prefix="roller_2_7"/>
-  <xacro:roller_gazebo_v0 prefix="roller_2_8"/>
-  <xacro:roller_gazebo_v0 prefix="roller_2_9"/>
-  <xacro:roller_gazebo_v0 prefix="roller_3_1"/>
-  <xacro:roller_gazebo_v0 prefix="roller_3_2"/>
-  <xacro:roller_gazebo_v0 prefix="roller_3_3"/>
-  <xacro:roller_gazebo_v0 prefix="roller_3_4"/>
-  <xacro:roller_gazebo_v0 prefix="roller_3_5"/>
-  <xacro:roller_gazebo_v0 prefix="roller_3_6"/>
-  <xacro:roller_gazebo_v0 prefix="roller_3_7"/>
-  <xacro:roller_gazebo_v0 prefix="roller_3_8"/>
-  <xacro:roller_gazebo_v0 prefix="roller_3_9"/>
-  <xacro:roller_gazebo_v0 prefix="roller_4_1"/>
-  <xacro:roller_gazebo_v0 prefix="roller_4_2"/>
-  <xacro:roller_gazebo_v0 prefix="roller_4_3"/>
-  <xacro:roller_gazebo_v0 prefix="roller_4_4"/>
-  <xacro:roller_gazebo_v0 prefix="roller_4_5"/>
-  <xacro:roller_gazebo_v0 prefix="roller_4_6"/>
-  <xacro:roller_gazebo_v0 prefix="roller_4_7"/>
-  <xacro:roller_gazebo_v0 prefix="roller_4_8"/>
-  <xacro:roller_gazebo_v0 prefix="roller_4_9"/>
-  <!-- Rollor -->
-  <xacro:roller_trans_v0 prefix="roller_1_1"/>
-  <xacro:roller_trans_v0 prefix="roller_1_2"/>
-  <xacro:roller_trans_v0 prefix="roller_1_3"/>
-  <xacro:roller_trans_v0 prefix="roller_1_4"/>
-  <xacro:roller_trans_v0 prefix="roller_1_5"/>
-  <xacro:roller_trans_v0 prefix="roller_1_6"/>
-  <xacro:roller_trans_v0 prefix="roller_1_7"/>
-  <xacro:roller_trans_v0 prefix="roller_1_8"/>
-  <xacro:roller_trans_v0 prefix="roller_1_9"/>
-  <xacro:roller_trans_v0 prefix="roller_2_1"/>
-  <xacro:roller_trans_v0 prefix="roller_2_2"/>
-  <xacro:roller_trans_v0 prefix="roller_2_3"/>
-  <xacro:roller_trans_v0 prefix="roller_2_4"/>
-  <xacro:roller_trans_v0 prefix="roller_2_5"/>
-  <xacro:roller_trans_v0 prefix="roller_2_6"/>
-  <xacro:roller_trans_v0 prefix="roller_2_7"/>
-  <xacro:roller_trans_v0 prefix="roller_2_8"/>
-  <xacro:roller_trans_v0 prefix="roller_2_9"/>
-  <xacro:roller_trans_v0 prefix="roller_3_1"/>
-  <xacro:roller_trans_v0 prefix="roller_3_2"/>
-  <xacro:roller_trans_v0 prefix="roller_3_3"/>
-  <xacro:roller_trans_v0 prefix="roller_3_4"/>
-  <xacro:roller_trans_v0 prefix="roller_3_5"/>
-  <xacro:roller_trans_v0 prefix="roller_3_6"/>
-  <xacro:roller_trans_v0 prefix="roller_3_7"/>
-  <xacro:roller_trans_v0 prefix="roller_3_8"/>
-  <xacro:roller_trans_v0 prefix="roller_3_9"/>
-  <xacro:roller_trans_v0 prefix="roller_4_1"/>
-  <xacro:roller_trans_v0 prefix="roller_4_2"/>
-  <xacro:roller_trans_v0 prefix="roller_4_3"/>
-  <xacro:roller_trans_v0 prefix="roller_4_4"/>
-  <xacro:roller_trans_v0 prefix="roller_4_5"/>
-  <xacro:roller_trans_v0 prefix="roller_4_6"/>
-  <xacro:roller_trans_v0 prefix="roller_4_7"/>
-  <xacro:roller_trans_v0 prefix="roller_4_8"/>
-  <xacro:roller_trans_v0 prefix="roller_4_9"/>
   <!-- ultrasound -->
   <xacro:zm_ultrasound prefix="1" parent="base_link" origin_x="${ul_left_front_x}" origin_y="${ul_left_front_y}"

File: zm_robot_description/urdf/zm_robot_roller.urdf.xacro (robot description, xacro)
@@ -1,8 +1,6 @@
 <?xml version="1.0"?>
 <robot xmlns:xacro="http://ros.org/wiki/xacro">
-  <xacro:include filename="$(find zm_robot_description)/urdf/zm_robot_roller.transmission.xacro"/>
-  <xacro:include filename="$(find zm_robot_description)/urdf/zm_robot_roller.gazebo"/>
   <xacro:macro name="zm_roller_v0" params="prefix parent origin_x origin_y rotation_x rotation_z">
-	<joint name="${prefix}_joint" type="continuous">
+	<joint name="${prefix}_joint" type="fixed">
 	  <parent link="${parent}"/>
 	  <child link="${prefix}"/>

File: zm_robot_description/urdf/zm_robot_ultrasound.urdf.xacro (robot description, xacro)
@@ -1,5 +1,4 @@
 <?xml version="1.0"?>
 <robot xmlns:xacro="http://ros.org/wiki/xacro">
-  <xacro:include filename="$(find zm_robot_description)/urdf/zm_robot_ultrasound.gazebo"/>
   <xacro:macro name="zm_ultrasound" params="prefix parent origin_x origin_y origin_z rotation_z">
 	<joint name="ultrasound_joint_${prefix}" type="fixed">

File: zm_robot_description/urdf/zm_robot_wheel_LF.urdf.xacro (robot description, xacro)
@@ -3,5 +3,5 @@
   <xacro:include filename="$(find zm_robot_description)/urdf/zm_robot_wheel.gazebo"/>
   <xacro:macro name="zm_wheel_v2" params="prefix parent origin_x origin_y rotation_x">
-	<joint name="wheel_joint_${prefix}" type="continuous">
+	<joint name="wheel_joint_${prefix}" type="fixed">
 	  <parent link="${parent}"/>
 	  <child link="wheel_${prefix}"/>

File: zm_robot_description/urdf/zm_robot_wheel_LR.urdf.xacro (robot description, xacro)
@@ -3,5 +3,5 @@
   <xacro:include filename="$(find zm_robot_description)/urdf/zm_robot_wheel.gazebo"/>
   <xacro:macro name="zm_wheel_v1" params="prefix parent origin_x origin_y rotation_x">
-	<joint name="wheel_joint_${prefix}" type="continuous">
+	<joint name="wheel_joint_${prefix}" type="fixed">
 	  <parent link="${parent}"/>
 	  <child link="wheel_${prefix}"/>

File: zm_robot_description/urdf/zm_robot_wheel_RF.urdf.xacro (robot description, xacro)
@@ -1,7 +1,6 @@
 <?xml version="1.0"?>
 <robot xmlns:xacro="http://ros.org/wiki/xacro">
-  <xacro:include filename="$(find zm_robot_description)/urdf/zm_robot_wheel.gazebo"/>
   <xacro:macro name="zm_wheel_v3" params="prefix parent origin_x origin_y rotation_x">
-	<joint name="wheel_joint_${prefix}" type="continuous">
+	<joint name="wheel_joint_${prefix}" type="fixed">
 	  <parent link="${parent}"/>
 	  <child link="wheel_${prefix}"/>

File: zm_robot_description/urdf/zm_robot_wheel_RR.urdf.xacro (robot description, xacro)
@@ -3,5 +3,5 @@
   <xacro:include filename="$(find zm_robot_description)/urdf/zm_robot_wheel.gazebo"/>
   <xacro:macro name="zm_wheel_v4" params="prefix parent origin_x origin_y rotation_x">
-	<joint name="wheel_joint_${prefix}" type="continuous">
+	<joint name="wheel_joint_${prefix}" type="fixed">
 	  <parent link="${parent}"/>
 	  <child link="wheel_${prefix}"/>
