Commit message: Fixed Imu link name

File: zm_robot_description/urdf/zm_robot.urdf.xacro (robot description, xacro)
@@ -168,9 +168,9 @@
   <joint name="IMU_joint " type="fixed">
     <parent link="base_link"/>
-    <child link="IMU_sensor"/>
+    <child link="imu_link"/>
     <origin xyz="0 0 0.08" rpy="0 0 0"/>
     <axis xyz="0 0 1"/>
   </joint>
-  <link name="IMU_sensor">
+  <link name="imu_link">
     <sensor name="imu" type="imu">
       <update_rate>30</update_rate>

File: zm_robot_description/urdf/zm_robot_wheel_LF.urdf.xacro (robot description, xacro)
@@ -1,5 +1,4 @@
 <?xml version="1.0"?>
 <robot xmlns:xacro="http://ros.org/wiki/xacro">
-  <xacro:include filename="$(find zm_robot_description)/urdf/zm_robot_wheel.gazebo"/>
   <xacro:macro name="zm_wheel_v2" params="prefix parent origin_x origin_y rotation_x">
 	<joint name="wheel_joint_${prefix}" type="fixed">

File: zm_robot_description/urdf/zm_robot_wheel_LR.urdf.xacro (robot description, xacro)
@@ -1,5 +1,4 @@
 <?xml version="1.0"?>
 <robot xmlns:xacro="http://ros.org/wiki/xacro">
-  <xacro:include filename="$(find zm_robot_description)/urdf/zm_robot_wheel.gazebo"/>
   <xacro:macro name="zm_wheel_v1" params="prefix parent origin_x origin_y rotation_x">
 	<joint name="wheel_joint_${prefix}" type="fixed">

File: zm_robot_description/urdf/zm_robot_wheel_RR.urdf.xacro (robot description, xacro)
@@ -1,5 +1,4 @@
 <?xml version="1.0"?>
 <robot xmlns:xacro="http://ros.org/wiki/xacro">
-  <xacro:include filename="$(find zm_robot_description)/urdf/zm_robot_wheel.gazebo"/>
   <xacro:macro name="zm_wheel_v4" params="prefix parent origin_x origin_y rotation_x">
 	<joint name="wheel_joint_${prefix}" type="fixed">
